Commit message: Tried to make URDF for KCG

File: kneed_compass_gait.urdf (robot description, URDF)
Before this commit: robot kneed_compass_gait, 6 links, 6 joints
Links:
- added link stance_hip, mass 1; visual cylinder length=1 radius=.01; visual sphere radius=.05
- added link swing_hip, mass 1; visual cylinder length=1 radius=.01; visual sphere radius=.05
Joints:
- removed joint body_on_stance_leg
- removed joint hip_pin
- added joint body_to_swing_hip: type continuous, parent swing_hip, child swing_leg, origin xyz=0 0 -1, axis 0 -1 0
- added joint stance_hip_to_body: type fixed, parent stance_hip, child body, origin xyz=0 0 1
- added joint stance_knee_joint: type fixed, parent stance_leg, child stance_hip, origin xyz=0 0 1, axis 0 -1 0
